File: pcb/onewire.kicad_sch (KiCad schematic)
At the start: 7 parts, among them J15 Conn_01x03, J16 Conn_01x03, J17 Screw_Terminal_01x03, Q1 BSS138, U1 DS18B20

Commit message: wip
Parts:
- J17: footprint Conn_ScrewTerminals:ED5553DS -> Conn_ScrewTerminals:CTB7000-3
Changed lines of the file:
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@@
 	(label "ONEWIRE_5V"
 		(at 173.99 114.3 0)
-		(fields_autoplaced yes)
 		(effects
 			(font
@@
 	(label "ONEWIRE_5V"
 		(at 76.2 160.02 0)
-		(fields_autoplaced yes)
 		(effects
 			(font
@@
 	(label "ONEWIRE_5V"
 		(at 114.3 63.5 0)
-		(fields_autoplaced yes)
 		(effects
 			(font
@@
 	(label "ONEWIRE_5V"
 		(at 76.2 109.22 0)
-		(fields_autoplaced yes)
 		(effects
 			(font
@@
 	(label "ONEWIRE_5V"
 		(at 76.2 134.62 0)
-		(fields_autoplaced yes)
 		(effects
 			(font
@@
 		(shape bidirectional)
 		(at 63.5 63.5 180)
-		(fields_autoplaced yes)
 		(effects
 			(font
@@
 			)
 		)
-		(property "Footprint" "Conn_ScrewTerminals:ED5553DS"
+		(property "Footprint" "Conn_ScrewTerminals:CTB7000-3"
 			(at 71.12 162.56 0)
 			(effects

Commit message: wip
Parts:
- removed J17: Screw_Terminal_01x03, Conn_ScrewTerminals:CTB7000-3, symbol Connector:Screw_Terminal_01x03
Changed lines of the file:
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@@
-	)
-	(label "ONEWIRE_5V"
-		(at 76.2 160.02 0)
-		(effects
-			(font
-				(size 1.27 1.27)
-			)
-			(justify left bottom)
-		)
 	)
 	(label "ONEWIRE_5V"
@@
 	)
 	(symbol
-		(lib_id "power:+5V")
-		(at 76.2 162.56 270)
-		(unit 1)
-		(exclude_from_sim no)
-		(in_bom yes)
-		(on_board yes)
-		(dnp no)
-		(fields_autoplaced yes)
-		(property "Reference" "#PWR039"
-			(at 72.39 162.56 0)
-			(effects
-				(font
-					(size 1.27 1.27)
-				)
-				(hide yes)
-			)
-		)
-		(property "Value" "+5V"
-			(at 80.01 162.5599 90)
-			(effects
-				(font
-					(size 1.27 1.27)
-				)
-				(justify left)
-			)
-		)
-		(property "Footprint" ""
-			(at 76.2 162.56 0)
-			(effects
-				(font
-					(size 1.27 1.27)
-				)
-				(hide yes)
-			)
-		)
-		(property "Datasheet" ""
-			(at 76.2 162.56 0)
-			(effects
-				(font
-					(size 1.27 1.27)
-				)
-				(hide yes)
-			)
-		)
-		(property "Description" "Power symbol creates a global label with name \"+5V\""
-			(at 76.2 162.56 0)
-			(effects
-				(font
-					(size 1.27 1.27)
-				)
-				(hide yes)
-			)
-		)
-		(pin "1"
-		)
-		(instances
-			(project "pico-plc"
-				(path "/fc9ff52a-d720-4efe-8661-3db6c88a54e4/41233123-d0bb-4504-988d-344ca09ddc46"
-					(reference "#PWR039")
-					(unit 1)
-				)
-			)
-		)
-	)
-	(symbol
 		(lib_id "power:+3V3")
 		(at 76.2 44.45 0)
@@
 	)
 	(symbol
-		(lib_id "Connector:Screw_Terminal_01x03")
-		(at 71.12 162.56 180)
-		(unit 1)
-		(exclude_from_sim no)
-		(in_bom yes)
-		(on_board yes)
-		(dnp no)
-		(fields_autoplaced yes)
-		(property "Reference" "J17"
-			(at 71.12 153.67 0)
-			(effects
-				(font
-					(size 1.27 1.27)
-				)
-			)
-		)
-		(property "Value" "Screw_Terminal_01x03"
-			(at 71.12 156.21 0)
-			(effects
-				(font
-					(size 1.27 1.27)
-				)
-			)
-		)
-		(property "Footprint" "Conn_ScrewTerminals:CTB7000-3"
-			(at 71.12 162.56 0)
-			(effects
-				(font
-					(size 1.27 1.27)
-				)
-				(hide yes)
-			)
-		)
-		(property "Datasheet" "~"
-			(at 71.12 162.56 0)
-			(effects
-				(font
-					(size 1.27 1.27)
-				)
-				(hide yes)
-			)
-		)
-		(property "Description" "Generic screw terminal, single row, 01x03, script generated (kicad-library-utils/schlib/autogen/connector/)"
-			(at 71.12 162.56 0)
-			(effects
-				(font
-					(size 1.27 1.27)
-				)
-				(hide yes)
-			)
-		)
-		(pin "3"
-		)
-		(pin "2"
-		)
-		(pin "1"
-		)
-		(instances
-			(project ""
-				(path "/fc9ff52a-d720-4efe-8661-3db6c88a54e4/41233123-d0bb-4504-988d-344ca09ddc46"
-					(reference "J17")
-					(unit 1)
-				)
-			)
-		)
-	)
-	(symbol
 		(lib_id "power:+5V")
 		(at 76.2 137.16 270)
@@
 					(unit 1)
 				)
-			)
-		)
-	)
-	(symbol
-		(lib_id "power:GND")
-		(at 76.2 165.1 90)
-		(unit 1)
-		(exclude_from_sim no)
-		(in_bom yes)
-		(on_board yes)
-		(dnp no)
-		(fields_autoplaced yes)
-		(property "Reference" "#PWR040"
-			(at 82.55 165.1 0)
-			(effects
-				(font
-					(size 1.27 1.27)
-				)
-				(hide yes)
-			)
-		)
-		(property "Value" "GND"
-			(at 80.01 165.0999 90)
-			(effects
-				(font
-					(size 1.27 1.27)
-				)
-				(justify right)
-			)
-		)
-		(property "Footprint" ""
-			(at 76.2 165.1 0)
-			(effects
-				(font
-					(size 1.27 1.27)
-				)
-				(hide yes)
-			)
-		)
-		(property "Datasheet" ""
-			(at 76.2 165.1 0)
-			(effects
-				(font
-					(size 1.27 1.27)
-				)
-				(hide yes)
-			)
-		)
-		(property "Description" "Power symbol creates a global label with name \"GND\" , ground"
-			(at 76.2 165.1 0)
-			(effects
-				(font
-					(size 1.27 1.27)
-				)
-				(hide yes)
-			)
-		)
-		(pin "1"
-		)
-		(instances
-			(project "pico-plc"
-				(path "/fc9ff52a-d720-4efe-8661-3db6c88a54e4/41233123-d0bb-4504-988d-344ca09ddc46"
-					(reference "#PWR040")
-					(unit 1)
-				)
