File: pcb/pico-plc.kicad_pcb (KiCad board)
At the start: 2 copper layers, 142.5 x 95.5 mm, 183 parts, among them J1 Conn_02x06_Odd_Even, J10 Screw_Terminal_01x02, J11 Screw_Terminal_01x02, J12 Conn_01x02, J13 Conn_01x02, J14 Conn_01x02, J15 Conn_01x03, J16 Conn_01x03, J17 Screw_Terminal_01x03, J18 Screw_Terminal_01x03, J19 Screw_Terminal_01x03, J2 Conn_01x06, J20 Screw_Terminal_01x03, J21 Screw_Terminal_01x03, J22 Screw_Terminal_01x03, J23 Screw_Terminal_01x03, J24 Screw_Terminal_01x03, J25 Screw_Terminal_01x03, J26 Screw_Terminal_01x02, J27 Screw_Terminal_01x02, J28 Screw_Terminal_01x02, J29 Screw_Terminal_01x02, J3 Conn_02x06_Odd_Even, J30 Screw_Terminal_01x02, J31 Screw_Terminal_01x02, J32 Screw_Terminal_01x02, J33 Screw_Terminal_01x02, J34 Screw_Terminal_01x02, J35 Conn_01x02, J36 Conn_01x02, J4 Screw_Terminal_01x02, J5 Conn_01x06, J6 Conn_01x06, J7 Screw_Terminal_01x02, J8 Conn_01x02, J9 Screw_Terminal_01x02, K1 Relay_SPDT, K2 Relay_SPDT, K3 Relay_SPDT, K4 Relay_SPDT, K5 Relay_SPDT, K6 Relay_SPDT, K7 Relay_SPDT, K8 Relay_SPDT, Q1 BSS138, Q10 NDS355AN, Q11 NDS355AN, Q12 NDS355AN, Q13 NDS355AN, Q14 NDS355AN, Q15 NDS355AN, Q2 BSS138, Q3 BSS138, Q4 BSS138, Q5 BSS138, Q6 BSS138, Q7 BSS138, Q8 NDS355AN, Q9 NDS355AN, SW1 Reset, SW2 Power Cycle, U1 DS18B20, U2 VO615A, U3 VO615A, U4 VO615A, U5 VO615A, U6 VO615A, U7 VO615A, U8 VO615A, U9 VO615A

Commit message: wip
Parts:
- J10, J11, J26, J27, J28, J29, J30, J31, J32, J33, J34, J4, J7, J9: footprint Conn_ScrewTerminals:ED5552DS -> Conn_ScrewTerminals:CTB7000-2
- J17, J18, J19, J20, J21, J22, J23, J24, J25: footprint Conn_ScrewTerminals:ED5553DS -> Conn_ScrewTerminals:CTB7000-3
- R17, R21, R25, R29, R33, R37, R41, R45: value 4k7 -> 10k
- moved J34 183.7 mm to (-73.3, 91.6), turned to 0 degrees
- moved J4 178.0 mm to (-73.3, 41.1), turned to 0 degrees
- moved J9 166.2 mm to (-73.3, 61.3), turned to 0 degrees
- moved J10 156.6 mm to (-73.3, 71.4), turned to 0 degrees
- moved J27 154.6 mm to (-47.1, 53.2), turned to 0 degrees
- moved J11 147.7 mm to (-73.3, 81.5), turned to 0 degrees
- moved J28 146.9 mm to (-47.1, 41.1), turned to 0 degrees
- moved J30 144.8 mm to (-60.2, 53.2), turned to 0 degrees
- moved J7 136.5 mm to (-73.3, 51.2), turned to 0 degrees
- moved J26 136.0 mm to (-20.9, 53.2), turned to 0 degrees
- moved J33 121.9 mm to (-60.2, 41.1), turned to 0 degrees
- moved J29 113.1 mm to (-20.9, 41.1), turned to 0 degrees
- moved J31 111.1 mm to (-34.0, 53.2), turned to 0 degrees
- moved J32 103.4 mm to (-34.0, 41.1), turned to 0 degrees
- moved J17 28.9 mm to (139.0, 20.3)
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Routing:
- net +5V: track 467.0 -> 575.9 mm, vias 14 -> 28
- net Net-(D9-A): track 17.1 -> 51.2 mm
- net Net-(D7-A): track 17.1 -> 51.2 mm
- net Net-(D5-A): track 17.1 -> 51.2 mm
- net Net-(D19-A): track 17.1 -> 51.2 mm
- net Net-(D13-A): track 17.1 -> 51.2 mm
- net Net-(D15-A): track 17.1 -> 51.2 mm
- net Net-(D11-A): track 17.1 -> 51.2 mm
- net /Relays/Relay 2/COM: track 24.1 -> 49.8 mm
- net /Relays/Relay 0/COM: track 24.1 -> 49.8 mm
- net /Relays/Relay 7/COM: track 24.1 -> 49.8 mm
- net /Relays/Relay 5/COM: track 24.1 -> 49.8 mm
- net /Relays/Relay 4/COM: track 24.1 -> 49.8 mm
- net /Relays/Relay 3/COM: track 24.1 -> 49.8 mm
- net /Relays/Relay 1/COM: track 24.1 -> 49.8 mm
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
Commit message: wip
Parts:
- moved J34 22.6 mm to (-52.3, 83.3)
Changed lines of the file:
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@@
 		)
 	)
+	(footprint "Conn_ScrewTerminals:CTB7000-2"
+		(layer "F.Cu")
+		(at -52.324 83.312)
+		(property "Reference" "J34"
+			(at 0 -5.5 0)
+			(unlocked yes)
+			(layer "F.SilkS")
+			(effects
+				(font
+					(size 1 1)
+					(thickness 0.1)
+				)
+			)
+		)
+		(property "Value" "Screw_Terminal_01x02"
+			(at 0 5.5 0)
+			(unlocked yes)
+			(layer "F.Fab")
+			(effects
+				(font
+					(size 1 1)
+					(thickness 0.15)
+				)
+			)
+		)
+		(property "Footprint" "Conn_ScrewTerminals:CTB7000-2"
+			(at 0 0 0)
+			(unlocked yes)
+			(layer "F.Fab")
+			(hide yes)
+			(effects
+				(font
+					(size 1 1)
+					(thickness 0.15)
+				)
+			)
+		)
+		(property "Datasheet" ""
+			(at 0 0 0)
+			(unlocked yes)
+			(layer "F.Fab")
+			(hide yes)
+			(effects
+				(font
+					(size 1 1)
+					(thickness 0.15)
+				)
+			)
+		)
+		(property "Description" "Generic screw terminal, single row, 01x02, script generated (kicad-library-utils/schlib/autogen/connector/)"
+			(at 0 0 0)
+			(unlocked yes)
+			(layer "F.Fab")
+			(hide yes)
+			(effects
+				(font
+					(size 1 1)
+					(thickness 0.15)
+				)
+			)
+		)
+		(property ki_fp_filters "TerminalBlock*:*")
+		(sheetname "Power")
+		(sheetfile "power.kicad_sch")
+		(attr through_hole)
+		(fp_line
+			(start -5 -4.5)
+			(end -5 4.5)
+			(stroke
+				(width 0.1)
+				(type default)
+			)
+			(layer "F.SilkS")
+		)
+		(fp_line
+			(start -5 -4.5)
+			(end 5 -4.5)
+			(stroke
+				(width 0.1)
+				(type default)
+			)
+			(layer "F.SilkS")
+		)
+		(fp_line
+			(start -5 3.5)
+			(end 5 3.5)
+			(stroke
+				(width 0.1)
+				(type default)
+			)
+			(layer "F.SilkS")
+		)
+		(fp_line
+			(start -5 4.5)
+			(end 5 4.5)
+			(stroke
+				(width 0.1)
+				(type default)
+			)
+			(layer "F.SilkS")
+		)
+		(fp_line
+			(start 0 -4.5)
+			(end 0 4.5)
+			(stroke
+				(width 0.1)
+				(type default)
+			)
+			(layer "F.SilkS")
+		)
+		(fp_line
+			(start 5 -4.5)
+			(end 5 4.5)
+			(stroke
+				(width 0.1)
+				(type default)
+			)
+			(layer "F.SilkS")
+		)
+		(fp_text user "${REFERENCE}"
+			(at 0 7 0)
+			(unlocked yes)
+			(layer "F.Fab")
+			(effects
+				(font
+					(size 1 1)
+					(thickness 0.15)
+				)
+			)
+		)
+		(pad "1" thru_hole roundrect
+			(at 2.5 0)
+			(size 3 3)
+			(drill 1.3)
+			(layers "*.Cu" "*.Mask")
+			(remove_unused_layers no)
+			(roundrect_rratio 0.1)
+			(net 3 "GND")
+			(pinfunction "Pin_1")
+			(pintype "passive")
+		)
+		(pad "2" thru_hole circle
+			(at -2.5 0)
+			(size 3 3)
+			(drill 1.3)
+			(layers "*.Cu" "*.Mask")
+			(remove_unused_layers no)
+			(net 8 "+5V")
+			(pinfunction "Pin_2")
+			(pintype "passive")
+		)
+	)
 	(footprint "Diode_SMD:D_SOD-123"
 		(layer "F.Cu")
@@
 		)
 	)
-	(footprint "Conn_ScrewTerminals:CTB7000-2"
-		(layer "F.Cu")
-		(at -73.31 91.635)
-		(property "Reference" "J34"
-			(at 0 -5.5 0)
-			(unlocked yes)
-			(layer "F.SilkS")
-			(effects
-				(font
-					(size 1 1)
-					(thickness 0.1)
-				)
-			)
-		)
-		(property "Value" "Screw_Terminal_01x02"
-			(at 0 5.5 0)
-			(unlocked yes)
-			(layer "F.Fab")
-			(effects
-				(font
-					(size 1 1)
-					(thickness 0.15)
-				)
-			)
-		)
-		(property "Footprint" "Conn_ScrewTerminals:CTB7000-2"
-			(at 0 0 0)
-			(unlocked yes)
-			(layer "F.Fab")
-			(hide yes)
-			(effects
-				(font
-					(size 1 1)
-					(thickness 0.15)
-				)
-			)
-		)
-		(property "Datasheet" ""
-			(at 0 0 0)
-			(unlocked yes)
-			(layer "F.Fab")
-			(hide yes)
-			(effects
-				(font
-					(size 1 1)
-					(thickness 0.15)
-				)
-			)
-		)
-		(property "Description" "Generic screw terminal, single row, 01x02, script generated (kicad-library-utils/schlib/autogen/connector/)"
-			(at 0 0 0)
-			(unlocked yes)
-			(layer "F.Fab")
-			(hide yes)
-			(effects
-				(font
-					(size 1 1)
-					(thickness 0.15)
-				)
-			)
-		)
-		(property ki_fp_filters "TerminalBlock*:*")
-		(sheetname "Power")
-		(sheetfile "power.kicad_sch")
-		(attr through_hole)
-		(fp_line
-			(start -5 -4.5)
-			(end -5 4.5)
-			(stroke
-				(width 0.1)
-				(type default)
-			)
-			(layer "F.SilkS")
-		)
-		(fp_line
-			(start -5 -4.5)
-			(end 5 -4.5)
-			(stroke
-				(width 0.1)
-				(type default)
-			)
-			(layer "F.SilkS")
-		)
-		(fp_line
-			(start -5 3.5)
-			(end 5 3.5)
-			(stroke
-				(width 0.1)
-				(type default)
-			)
-			(layer "F.SilkS")
-		)
-		(fp_line
-			(start -5 4.5)
-			(end 5 4.5)
-			(stroke
-				(width 0.1)
-				(type default)
-			)
-			(layer "F.SilkS")
-		)
-		(fp_line
-			(start 0 -4.5)
-			(end 0 4.5)
-			(stroke
-				(width 0.1)
-				(type default)
-			)
-			(layer "F.SilkS")
-		)
-		(fp_line
-			(start 5 -4.5)
-			(end 5 4.5)
-			(stroke
-				(width 0.1)
-				(type default)
-			)
-			(layer "F.SilkS")
-		)
-		(fp_text user "${REFERENCE}"
-			(at 0 7 0)
-			(unlocked yes)
-			(layer "F.Fab")
-			(effects
-				(font
-					(size 1 1)
-					(thickness 0.15)
-				)
-			)
-		)
-		(pad "1" thru_hole roundrect
-			(at 2.5 0)
-			(size 3 3)
-			(drill 1.3)
-			(layers "*.Cu" "*.Mask")
-			(remove_unused_layers no)
-			(roundrect_rratio 0.1)
-			(net 3 "GND")
-			(pinfunction "Pin_1")
-			(pintype "passive")
-		)
-		(pad "2" thru_hole circle
-			(at -2.5 0)
-			(size 3 3)
-			(drill 1.3)
-			(layers "*.Cu" "*.Mask")
-			(remove_unused_layers no)
-			(net 8 "+5V")
-			(pinfunction "Pin_2")
-			(pintype "passive")
-		)
-	)
 	(footprint "Connector_PinHeader_2.54mm:PinHeader_1x02_P2.54mm_Vertical"
 		(layer "F.Cu")
@@
 		(fp_arc
 			(start 10.579676 25.189937)
-			(mid 10.357949 25.493953)
+			(mid 10.357946 25.493957)
 			(end 10 25.61)
 			(stroke

Commit message: wip
Routing:
- net +5V: track 575.9 -> 469.7 mm
- net /IO20: track 16.8 -> 5.10 mm
- net /Power/Power In: track 9.35 -> 0.00 mm
- net /IO19: track 15.7 -> 7.64 mm
- net +3V3: track 277.4 -> 269.8 mm, vias 17 -> 16
- net /IO6: track 108.8 -> 101.7 mm
- net /IO7: track 122.5 -> 117.0 mm
- net /IO16: track 52.1 -> 48.5 mm
- net Net-(D3-K): track 2.74 -> 0.00 mm
- net Net-(D2-K): track 2.74 -> 0.00 mm
- net /IO17: track 38.1 -> 35.4 mm
- net /IO21: track 31.2 -> 29.3 mm
- net /IO18: track 27.1 -> 25.5 mm
- net /OneWire/ONEWIRE_5V: track 42.2 -> 40.9 mm
- net /Opto Inputs/Input 7/SIG: track 4.82 -> 3.92 mm
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
Commit message: wip
Parts:
- removed J10, J11, J34, J4, J9: Screw_Terminal_01x02, Conn_ScrewTerminals:CTB7000-2
- H1, H2, H3, H4: footprint MountingHole:MountingHole_3.2mm_M3 -> MountingHole:MountingHole_3.2mm_M3_Pad_Via
- moved J7 159.2 mm to (27.9, 174.0), turned to -90 degrees
- moved D2 105.0 mm to (54.4, 175.5)
- moved R1 104.5 mm to (50.3, 175.0)
- moved D3 101.1 mm to (55.6, 163.3)
- moved R2 100.6 mm to (50.5, 162.8)
- moved J12 90.0 mm to (73.0, 172.6)
- moved J13 90.0 mm to (81.9, 172.6)
- moved J14 90.0 mm to (90.8, 172.6)
- moved J35 90.0 mm to (99.7, 172.6)
- moved J36 90.0 mm to (108.6, 172.6)
- moved J8 82.3 mm to (29.1, 157.3)
- moved D1 82.3 mm to (25.9, 150.3)
- moved J30 48.7 mm to (-21.6, 23.6)
- moved J27 32.2 mm to (-34.7, 23.6)
- moved J26 32.1 mm to (-47.8, 35.7)
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Routing:
- net +5V: track 469.7 -> 432.1 mm
- net /OneWire/ONEWIRE_5V: track 40.9 -> 20.9 mm

Commit message: wip
Parts:
- moved J26 201.0 mm to (127.0, -63.5), turned to 180 degrees
- moved J27 174.2 mm to (116.2, -63.5), turned to 180 degrees
- moved J31 164.2 mm to (73.0, -63.5), turned to 180 degrees
- moved J29 162.9 mm to (94.6, -63.5), turned to 180 degrees
- moved J28 161.1 mm to (105.4, -63.5), turned to 180 degrees
- moved D12 151.2 mm to (275.0, 94.0)
- moved D13 151.2 mm to (275.0, 96.5)
- moved K8 151.2 mm to (324.3, 102.4)
- moved Q12 151.2 mm to (287.1, 95.9)
- moved R29 151.2 mm to (267.4, 94.6)
- moved R34 151.2 mm to (287.1, 92.7)
- moved R35 151.2 mm to (278.8, 94.6)
- moved D14 151.2 mm to (291.5, 94.0)
- moved D15 151.2 mm to (291.5, 96.5)
- moved D16 151.2 mm to (308.1, 94.0)
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Routing:
- net +5V: track 432.1 -> 333.9 mm, vias 28 -> 14
- net +3V3: track 269.8 -> 216.5 mm, vias 16 -> 8
- net /IO16: track 48.5 -> 14.2 mm
- net Net-(D7-A): track 51.2 -> 17.1 mm
- net Net-(D11-A): track 51.2 -> 17.1 mm
- net Net-(D19-A): track 51.2 -> 17.1 mm
- net Net-(D9-A): track 51.2 -> 17.1 mm
- net Net-(D5-A): track 51.2 -> 17.1 mm
- net Net-(D13-A): track 51.2 -> 17.1 mm
- net Net-(D15-A): track 51.2 -> 17.1 mm
- net /Relays/Relay 0/COM: track 49.8 -> 24.8 mm
- net /Relays/Relay 2/COM: track 49.8 -> 24.8 mm
- net /Relays/Relay 5/COM: track 49.8 -> 24.8 mm
- net /Relays/Relay 4/COM: track 49.8 -> 24.8 mm
- net /Relays/Relay 3/COM: track 49.8 -> 24.8 mm
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Other:
- board size 142.5 x 95.5 mm -> 284.1 x 95.5 mm
- board text added: "+ve"
- board text added: "-ve"
- board text removed: "COM"

Commit message: wip
Parts:
- removed J12, J13, J14, J35, J36: Conn_01x02, Connector_PinHeader_2.54mm:PinHeader_1x02_P2.54mm_Vertical
- moved K8 172.9 mm to (151.5, 102.5)
- moved D12 172.9 mm to (102.2, 94.0)
- moved D13 172.9 mm to (102.2, 96.6)
- moved D14 172.9 mm to (118.7, 94.0)
- moved D15 172.9 mm to (118.7, 96.6)
- moved D16 172.9 mm to (135.2, 94.0)
- moved D17 172.9 mm to (135.2, 96.6)
- moved D18 172.9 mm to (151.7, 94.0)
- moved D19 172.9 mm to (151.7, 96.6)
- moved D4 172.9 mm to (36.1, 94.0)
- moved D5 172.9 mm to (36.1, 96.6)
- moved D6 172.9 mm to (52.6, 94.0)
- moved D7 172.9 mm to (52.6, 96.6)
- moved D8 172.9 mm to (69.1, 94.0)
- moved D9 172.9 mm to (69.1, 96.6)
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Routing:
- net /IO7: track 117.0 -> 13.3 mm, vias 1 -> 0
- net /IO6: track 101.7 -> 14.4 mm, vias 1 -> 0
- net +3V3: track 216.5 -> 287.1 mm, vias 8 -> 15
- net /IO8: track 102.8 -> 133.5 mm
- net /IO9: track 92.9 -> 119.7 mm
- net /IO10: track 80.5 -> 103.4 mm
- net /IO22: track 32.1 -> 11.5 mm
- net /IO11: track 70.7 -> 89.6 mm
- net +5V: track 333.9 -> 315.9 mm
- net /IO12: track 60.9 -> 75.8 mm
- net /IO13: track 51.0 -> 62.0 mm
- net /OneWire/ONEWIRE_5V: track 33.0 -> 23.1 mm
- net /IO14: track 38.7 -> 45.7 mm
- net /IO15: track 29.1 -> 31.4 mm
Other:
- board size 284.1 x 95.5 mm -> 221.1 x 103 mm
- board text added: "2025-02-14"
- board text removed: "2024-10-11"
- board text removed: "Aux. Power Out"

Commit message: wip
Parts:
- removed J17: Screw_Terminal_01x03, Conn_ScrewTerminals:CTB7000-3
- removed SW1: Reset, Button_Switch_SMD:SW_Push_1P1T_NO_CK_KMR2
- removed SW2: Power Cycle, Button_Switch_SMD:SW_Push_1P1T_NO_CK_KMR2
- added J12: Screw_Terminal_01x02, Conn_ScrewTerminals:CTB7000-2, F.Cu at (73.7, 166.4)
- added J13: Screw_Terminal_01x02, Conn_ScrewTerminals:CTB7000-2, F.Cu at (73.7, 176.5)
- moved D2 168.1 mm to (203.8, 98.6)
- moved R2 168.1 mm to (200.0, 85.9)
- moved D3 168.1 mm to (205.1, 86.5)
- moved R1 168.1 mm to (199.8, 98.1)
- moved J16 108.3 mm to (213.4, 118.7)
- moved J15 108.3 mm to (213.4, 114.9)
- moved J7 85.5 mm to (-9.53, 97.2)
- moved H2 32.0 mm to (42.0, 46.0)
- moved H3 32.0 mm to (42.0, 125.0)
- moved D22 14.0 mm to (105.0, 66.0)
- moved R65 14.0 mm to (130.2, 66.7)
- moved R68 14.0 mm to (97.8, 66.7)
- moved R59 14.0 mm to (74.9, 53.3)
- moved R61 14.0 mm to (64.1, 53.3)
- moved R63 14.0 mm to (53.3, 53.3)
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Routing:
- net +3V3: track 287.1 -> 17.8 mm, vias 15 -> 0
- net +5V: track 315.9 -> 141.9 mm
- net /IO8: track 133.5 -> 22.3 mm
- net /IO9: track 119.7 -> 20.7 mm
- net /IO10: track 103.4 -> 19.1 mm
- net /IO11: track 89.6 -> 17.6 mm
- net /IO12: track 75.8 -> 16.0 mm
- net /IO13: track 62.0 -> 14.5 mm
- net /OneWire/ONEWIRE_5V: track 23.1 -> 0.00 mm
- net /3V3_EN: track 17.3 -> 3.17 mm
- net /IO15: track 31.4 -> 17.5 mm
- net /IO14: track 45.7 -> 31.7 mm
- net /RUN: track 15.0 -> 3.17 mm
- net /IO22: track 11.5 -> 8.60 mm
- net GND: vias 26 -> 24
Other:
- board size 221.1 x 103 mm -> 154.5 x 95.5 mm
- board text removed: "Pwr. Cycle"
- board text removed: "Reset"

Commit message: wip
Parts:
- moved REF** 165.4 mm to (42.5, 111.1)
- moved J13 97.3 mm to (86.4, 80.0), turned to 90 degrees
- moved J16 90.0 mm to (246.4, 35.1)
- moved J15 90.0 mm to (246.4, 31.2)
- moved J12 86.5 mm to (76.8, 80.0), turned to -90 degrees
- moved D1 78.2 mm to (52.7, 76.8)
- moved J8 77.6 mm to (52.1, 83.2)
- moved J7 57.1 mm to (45.1, 80.6)
- moved D3 18.9 mm to (186.7, 90.8)
- moved R2 17.0 mm to (186.7, 96.5), turned to -90 degrees
- moved D2 16.0 mm to (189.9, 90.8), turned to 90 degrees
- moved R1 10.0 mm to (189.9, 96.5)
Routing:
- net /IO8: track 22.3 -> 119.6 mm
- net /IO9: track 20.7 -> 105.7 mm
- net /IO10: track 19.1 -> 89.4 mm
- net /IO11: track 17.6 -> 75.6 mm
- net /IO12: track 16.0 -> 61.8 mm
- net /IO13: track 14.5 -> 48.0 mm
- net /IO22: track 8.60 -> 0.86 mm
Other:
- outline, holes or cut-outs redrawn
