File: pcb/pico-plc.kicad_pcb (KiCad board)
At the start: 2 copper layers, 154.5 x 95.5 mm, 172 parts, among them J1 Conn_02x06_Odd_Even, J12 Screw_Terminal_01x02, J13 Screw_Terminal_01x02, J15 Conn_01x03, J16 Conn_01x03, J18 Screw_Terminal_01x03, J19 Screw_Terminal_01x03, J2 Conn_01x06, J20 Screw_Terminal_01x03, J21 Screw_Terminal_01x03, J22 Screw_Terminal_01x03, J23 Screw_Terminal_01x03, J24 Screw_Terminal_01x03, J25 Screw_Terminal_01x03, J26 Screw_Terminal_01x02, J27 Screw_Terminal_01x02, J28 Screw_Terminal_01x02, J29 Screw_Terminal_01x02, J3 Conn_02x06_Odd_Even, J30 Screw_Terminal_01x02, J31 Screw_Terminal_01x02, J32 Screw_Terminal_01x02, J33 Screw_Terminal_01x02, J5 Conn_01x06, J6 Conn_01x06, J7 Screw_Terminal_01x02, J8 Conn_01x02, K1 Relay_SPDT, K2 Relay_SPDT, K3 Relay_SPDT, K4 Relay_SPDT, K5 Relay_SPDT, K6 Relay_SPDT, K7 Relay_SPDT, K8 Relay_SPDT, Q1 BSS138, Q10 NDS355AN, Q11 NDS355AN, Q12 NDS355AN, Q13 NDS355AN, Q14 NDS355AN, Q15 NDS355AN, Q2 BSS138, Q3 BSS138, Q4 BSS138, Q5 BSS138, Q6 BSS138, Q7 BSS138, Q8 NDS355AN, Q9 NDS355AN, U1 DS18B20, U2 VO615A, U3 VO615A, U4 VO615A, U5 VO615A, U6 VO615A, U7 VO615A, U8 VO615A, U9 VO615A

Commit message: wip
Parts:
- moved J15 131.8 mm to (126.4, 85.7), turned to 180 degrees
- moved J16 126.8 mm to (130.2, 85.7), turned to 180 degrees
- moved U1 94.9 mm to (116.4, 86.4), turned to 90 degrees
- moved R3 87.5 mm to (137.8, 73.7), turned to -90 degrees
- moved Q1 87.5 mm to (134.0, 73.7), turned to 0 degrees
- moved R4 87.5 mm to (130.2, 73.7), turned to -90 degrees
Routing:
- net +5V: track 329.8 -> 475.8 mm
- net +3V3: track 230.2 -> 293.7 mm, vias 14 -> 15
- net /IO22: track 2.89 -> 31.5 mm
- net /OneWire/ONEWIRE_5V: track 3.29 -> 30.6 mm
- net GND: vias 24 -> 32
Other:
- board text added: "2025-02-16"
- board text added: "Aux. Power Out"
- board text removed: "2025-02-14"

Commit message: wip
Routing:
- net /OneWire/ONEWIRE_5V: track 30.6 -> 29.9 mm
Changed lines of the file:
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@@
 			(disableapertmacros no)
 			(usegerberextensions yes)
-			(usegerberattributes yes)
-			(usegerberadvancedattributes yes)
+			(usegerberattributes no)
+			(usegerberadvancedattributes no)
 			(creategerberjobfile no)
 			(dashed_line_dash_ratio 12.000000)
@@
 		(tags "Through hole pin header THT 1x03 2.54mm single row")
 		(property "Reference" "J15"
-			(at 0 -2.33 360)
+			(at 0 -2.33 0)
 			(layer "F.SilkS")
 			(effects
@@
 		)
 		(property "Value" "Conn_01x03"
-			(at 0 7.41 360)
+			(at 0 7.41 0)
 			(layer "F.Fab")
 			(effects
@@
 		(tags "Through hole pin header THT 1x03 2.54mm single row")
 		(property "Reference" "J16"
-			(at 0 -2.33 360)
+			(at 0 -2.33 0)
 			(layer "F.SilkS")
 			(effects
@@
 		)
 		(property "Value" "Conn_01x03"
-			(at 0 7.41 360)
+			(at 0 7.41 0)
 			(layer "F.Fab")
 			(effects
@@
 		(tags "resistor handsolder")
 		(property "Reference" "R3"
-			(at -2.54 0 360)
+			(at -2.54 0 0)
 			(layer "F.SilkS")
 			(effects
@@
 		(tags "Raspberry Pi Pico module usb pcb antenna handsolder")
 		(property "Reference" "A1"
-			(at 11.7475 24.765 -90)
+			(at 8.89 27.305 270)
 			(unlocked yes)
 			(layer "F.SilkS")
@@
 					(thickness 0.15)
 				)
-				(justify left)
 			)
 		)
@@
 		(fp_arc
 			(start 10.579676 25.189937)
-			(mid 10.357949 25.493953)
+			(mid 10.357946 25.493957)
 			(end 10 25.61)
 			(stroke
@@
 		(tags "SOT TO_SOT_SMD")
 		(property "Reference" "Q1"
-			(at 0 -2.4 360)
+			(at 0 -2.4 0)
 			(layer "F.SilkS")
 			(effects
@@
 		)
 		(property "Value" "BSS138"
-			(at 0 2.4 360)
+			(at 0 2.4 0)
 			(layer "F.Fab")
 			(effects
@@
 		)
 		(fp_text user "${REFERENCE}"
-			(at 0 0 360)
+			(at 0 0 0)
 			(layer "F.Fab")
 			(effects
@@
 	)
 	(segment
-		(start 189.205 53.335)
-		(end 189.205 50.775)
+		(start 189.205 51.35419)
+		(end 187.38081 49.53)
 		(width 0.35)
 		(layer "F.Cu")
@@
 	)
 	(segment
-		(start 186.974186 49.53)
-		(end 181.61 49.53)
-		(width 0.35)
-		(layer "F.Cu")
-		(net 7)
-	)
-	(segment
 		(start 190.5 61.595)
 		(end 190.5 54.63)
@@
 	)
 	(segment
-		(start 188.219186 50.775)
-		(end 186.974186 49.53)
+		(start 189.205 53.335)
+		(end 189.205 51.35419)
 		(width 0.35)
 		(layer "F.Cu")
@@
 	)
 	(segment
-		(start 189.205 50.775)
-		(end 188.219186 50.775)
+		(start 187.38081 49.53)
+		(end 181.61 49.53)
 		(width 0.35)
 		(layer "F.Cu")
@@
 	)
 	(segment
-		(start 126.365 80.645)
-		(end 127 80.645)
-		(width 0.35)
-		(layer "F.Cu")
-		(net 66)
-	)
-	(segment
 		(start 130.175 74.66)
 		(end 131.175 73.66)
@@
 	)
 	(segment
-		(start 127 80.645)
-		(end 127.015 80.63)
-		(width 0.35)
-		(layer "F.Cu")
-		(net 66)
-	)
-	(segment
 		(start 130.175 80.63)
 		(end 130.175 74.66)
@@
 	)
 	(segment
-		(start 55.165 100.52)
-		(end 55.2325 100.4525)
-		(width 2.5)
-		(layer "F.Cu")
-		(net 84)
-	)
-	(segment
 		(start 55.2325 100.4525)
 		(end 55.2325 125.095)
@@
 	)
 	(segment
-		(start 71.675 100.52)
-		(end 71.7425 100.4525)
-		(width 2.5)
-		(layer "F.Cu")
-		(net 86)
-	)
-	(segment
 		(start 71.7425 100.4525)
 		(end 71.7425 125.095)
@@
 	)
 	(segment
-		(start 88.185 100.52)
-		(end 88.2525 100.4525)
-		(width 2.5)
-		(layer "F.Cu")
-		(net 91)
-	)
-	(segment
 		(start 88.2525 125.095)
 		(end 88.185 125.1625)
@@
 	)
 	(segment
-		(start 104.695 100.52)
-		(end 104.7625 100.4525)
-		(width 2.5)
-		(layer "F.Cu")
-		(net 94)
-	)
-	(segment
 		(start 104.7625 125.095)
 		(end 104.695 125.1625)
@@
 	)
 	(segment
-		(start 121.205 100.52)
-		(end 121.2725 100.4525)
-		(width 2.5)
-		(layer "F.Cu")
-		(net 97)
-	)
-	(segment
 		(start 121.2725 125.095)
 		(end 121.205 125.1625)
@@
 	)
 	(segment
-		(start 137.715 100.52)
-		(end 137.7825 100.4525)
-		(width 2.5)
-		(layer "F.Cu")
-		(net 99)
-	)
-	(segment
 		(start 137.7825 125.095)
 		(end 137.715 125.1625)
@@
 	)
 	(segment
-		(start 154.225 100.52)
-		(end 154.2925 100.4525)
-		(width 2.5)
-		(layer "F.Cu")
-		(net 101)
-	)
-	(segment
 		(start 154.2925 100.4525)
 		(end 154.2925 125.095)
@@
 	)
 	(segment
-		(start 170.735 100.52)
-		(end 170.8025 100.4525)
-		(width 2.5)
-		(layer "F.Cu")
-		(net 106)
-	)
-	(segment
