File: pcb/general_io.kicad_sch (KiCad schematic)
At the start: 5 parts, among them J1 Conn_02x06_Odd_Even, J2 Conn_01x06, J3 Conn_02x06_Odd_Even, J5 Conn_01x06, J6 Conn_01x06

Commit message: New board revision
Parts:
- removed J3: Conn_02x06_Odd_Even, Connector_PinHeader_2.54mm:PinHeader_2x06_P2.54mm_Vertical, symbol Connector_Generic:Conn_02x06_Odd_Even
- removed J5, J6: Conn_01x06, Connector_PinHeader_2.54mm:PinHeader_1x06_P2.54mm_Vertical, symbol Connector_Generic:Conn_01x06
Connections:
- net IO0 renamed IO_A
- net IO1 renamed IO_B
- net IO2 renamed IO_C
- net IO3 renamed IO_D
- net IO4 renamed IO_E
- net IO5 renamed IO_F
Other:
- removed sheet Configurable Level Shifter IO0
- removed sheet Configurable Level Shifter IO1
- removed sheet Configurable Level Shifter IO2
- removed sheet Configurable Level Shifter IO3
- removed sheet Configurable Level Shifter IO4
- removed sheet Configurable Level Shifter IO5
