File: pcb/opto_input.kicad_sch (KiCad schematic)
At the start: 6 parts, among them J26 Screw_Terminal_01x02, U2 VO615A

Commit message: New board revision
Parts:
- U2: footprint Package_DIP:SMDIP-4_W7.62mm -> Package_DIP:SMDIP-4_W9.53mm
Changed lines of the file:
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@@
 			)
 		)
-		(property "Footprint" "Package_DIP:SMDIP-4_W7.62mm"
+		(property "Footprint" "Package_DIP:SMDIP-4_W9.53mm"
 			(at 147.32 78.74 0)
 			(effects
