File: pcb/power.kicad_sch (KiCad schematic)
At the start: 17 parts, among them J10 Screw_Terminal_01x02, J11 Screw_Terminal_01x02, J12 Conn_01x02, J13 Conn_01x02, J14 Conn_01x02, J34 Screw_Terminal_01x02, J35 Conn_01x02, J36 Conn_01x02, J4 Screw_Terminal_01x02, J7 Screw_Terminal_01x02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

Commit message: wip
Parts:
- J10, J11, J34, J4, J7, J9: footprint Conn_ScrewTerminals:ED5552DS -> Conn_ScrewTerminals:CTB7000-2
Changed lines of the file:
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@@
 	(label "Power In"
 		(at 203.2 63.5 90)
-		(fields_autoplaced yes)
 		(effects
 			(font
@@
 			)
 		)
-		(property "Footprint" "Conn_ScrewTerminals:ED5552DS"
+		(property "Footprint" "Conn_ScrewTerminals:CTB7000-2"
 			(at 71.12 50.8 0)
 			(effects
@@
 			)
 		)
-		(property "Footprint" "Conn_ScrewTerminals:ED5552DS"
+		(property "Footprint" "Conn_ScrewTerminals:CTB7000-2"
 			(at 71.12 127 0)
 			(effects
@@
 			)
 		)
-		(property "Footprint" "Conn_ScrewTerminals:ED5552DS"
+		(property "Footprint" "Conn_ScrewTerminals:CTB7000-2"
 			(at 71.12 152.4 0)
 			(effects
@@
 			)
 		)
-		(property "Footprint" "Conn_ScrewTerminals:ED5552DS"
+		(property "Footprint" "Conn_ScrewTerminals:CTB7000-2"
 			(at 71.12 101.6 0)
 			(effects
@@
 			)
 		)
-		(property "Footprint" "Conn_ScrewTerminals:ED5552DS"
+		(property "Footprint" "Conn_ScrewTerminals:CTB7000-2"
 			(at 71.12 76.2 0)
 			(effects
@@
 			)
 		)
-		(property "Footprint" "Conn_ScrewTerminals:ED5552DS"
+		(property "Footprint" "Conn_ScrewTerminals:CTB7000-2"
 			(at 185.42 53.34 0)
 			(effects

Commit message: wip
Parts:
- removed J10, J11, J34, J4, J9: Screw_Terminal_01x02, Conn_ScrewTerminals:CTB7000-2, symbol Connector:Screw_Terminal_01x02

Commit message: wip
Parts:
- removed J14, J35, J36: Conn_01x02, Connector_PinHeader_2.54mm:PinHeader_1x02_P2.54mm_Vertical, symbol Connector_Generic:Conn_01x02
- J12, J13: value Conn_01x02 -> Screw_Terminal_01x02; footprint Connector_PinHeader_2.54mm:PinHeader_1x02_P2.54mm_Vertical -> Conn_ScrewTerminals:CTB7000-2; symbol Connector_Generic:Conn_01x02 -> Connector:Screw_Terminal_01x02

Commit message: wip
Connections:
- net +5V: now also J13.1 (Pin_1); no longer J13.2 (Pin_2)
- net GND: now also J13.2 (Pin_2); no longer J13.1 (Pin_1)

Commit message: New board revision
Parts:
- removed J12, J13: Screw_Terminal_01x02, Conn_ScrewTerminals:CTB7000-2, symbol Connector:Screw_Terminal_01x02
